Commit message: r2d2 moving

File: src/my_r2d2/urdf/r2d2.urdf (robot description, URDF)
Before this commit: robot r2d2, 16 links, 15 joints
Links:
- added link base_footprint
Joints:
- added joint base_to_base_footprint: type fixed, parent base_link, child base_footprint, origin xyz=0 0 -0.3

File: src/my_r2d2/urdf/r2d2.urdf.xacro (robot description, xacro)
@@ -12,4 +12,6 @@
   <xacro:property name="width" value=".2" />
   <xacro:property name="bodylen" value=".6" />
+  <xacro:property name="wheelRadius" value="0.035" />
+  <xacro:property name="footBaseThickness" value="0.1" />
   <xacro:macro name="default_inertial" params="mass">
       <inertial>
@@ -34,4 +36,11 @@
     <xacro:default_inertial mass="10"/>
   </link>
+  <link name="base_footprint">
+  </link>
+  <joint name="base_to_base_footprint" type="fixed">
+    <parent link="base_footprint"/>
+    <child link="base_link"/>
+    <origin xyz="0 0 ${+(bodylen/2)+(wheelRadius*2)+footBaseThickness}"/>
+  </joint>
   <link name="right_leg">
     <visual>
@@ -51,5 +60,5 @@
     <visual>
       <geometry>
-        <box size="0.4 .1 .1"/>
+        <box size="0.4 ${footBaseThickness} ${footBaseThickness}"/>
       </geometry>
       <material name="white"/>
@@ -65,5 +74,5 @@
       <origin rpy="1.57075 0 0" xyz="0 0 0"/>
       <geometry>
-        <cylinder length="0.1" radius="0.035"/>
+        <cylinder length="0.1" radius="${wheelRadius}"/>
       </geometry>
       <material name="black"/>
@@ -81,5 +90,5 @@
       <origin rpy="1.57075 0 0" xyz="0 0 0"/>
       <geometry>
-        <cylinder length="0.1" radius="0.035"/>
+        <cylinder length="0.1" radius="${wheelRadius}"/>
       </geometry>
       <material name="black"/>
@@ -109,5 +118,5 @@
     <visual>
       <geometry>
-        <box size="0.4 .1 .1"/>
+        <box size="0.4 ${footBaseThickness} ${footBaseThickness}"/>
       </geometry>
       <material name="white"/>
