Commit message: camera

File: src/my_r2d2/urdf/r2d2.urdf.xacro (robot description, xacro)
@@ -247,4 +247,11 @@
     </visual>
   </link>
+  <link name="eye">
+  </link>
+  <joint name="eye_to_box" type="fixed">
+    <parent link="box"/>
+    <child link="eye"/>
+    <origin rpy="1.57 3.14 1.57" xyz="0 0 0"/>
+  </joint>
   <joint name="tobox" type="fixed">
     <parent link="head"/>
